File: layouts/default/default.kicad_pcb (KiCad board)
At the start: 2 copper layers, 13 parts

Commit message: initial build, migrating to V6
Parts:
- added C13: 100nF ±10% 50V X7R, atopile:C0603-bd72f6, F.Cu at (0.00, -50.0)
- added C14: 100nF ±10% 16V X7R, atopile:C0402-b3ef17, F.Cu at (0.00, -120.0)
- added C15: 100nF ±10% 16V X7R, atopile:C0402-b3ef17, F.Cu at (0.00, -110.0)
- added C16: 100nF ±10% 16V X7R, atopile:C0402-b3ef17, F.Cu at (0.00, -130.0)
- added C17: 100nF ±10% 50V X7R, atopile:C0603-bd72f6, F.Cu at (0.00, 0.00)
- added C18: 100nF ±10% 16V X7R, atopile:C0402-b3ef17, F.Cu at (0.00, -150.0)
- added C19: 100nF ±10% 16V X7R, atopile:C0402-b3ef17, F.Cu at (0.00, -60.0)
- added C20: 100nF ±10% 16V X7R, atopile:C0402-b3ef17, F.Cu at (0.00, -80.0)
- added C21: 100nF ±10% 50V X7R, atopile:C0603-bd72f6, F.Cu at (0.00, -140.0)
- added C22: 100nF ±10% 16V X7R, atopile:C0402-b3ef17, F.Cu at (0.00, -100.0)
- added C23: 100nF ±10% 16V X7R, atopile:C0402-b3ef17, F.Cu at (0.00, -70.0)
- added C24: 100nF ±10% 16V X7R, atopile:C0402-b3ef17, F.Cu at (0.00, -40.0)
- added L1: , atopile:L0603-9cac2b, F.Cu at (0.00, -10.0)
- added R1: 0Ω 50mW, atopile:R0201-27027e, F.Cu at (0.00, -20.0)
- added R2: 1kΩ ±1% 62.5mW, atopile:R0402-56259e, F.Cu at (0.00, -30.0)
- added R3: 0Ω 50mW, atopile:R0201-27027e, F.Cu at (0.00, -90.0)
Connections:
- net ETH_PHY_RXN renamed ETH_RN
- net ETH_PHY_RXP renamed ETH_RP
- net ETH_PHY_TXN renamed ETH_TN
- net ETH_PHY_TXP renamed ETH_TP
- net SDMMC0_DET_GPIO3_A1_u renamed SDMMC_DET
- C1 pad 1: C5-net-1 -> hv-2
- C1 pad 2: C5-net -> gnd
- C10 pad 1: C20-net -> hv-2
- C10 pad 2: C20-net-1 -> gnd
- C11 pad 1: C21-net-1 -> hv-2
- C11 pad 2: C21-net -> gnd
- C12 pad 1: C22-net -> hv-2
- C12 pad 2: C22-net-1 -> gnd
- C2 pad 1: C6-net -> hv-2
- C2 pad 2: C6-net-1 -> gnd
- C3 pad 1: C7-net-1 -> hv-2
- C3 pad 2: C7-net -> gnd
- C4 pad 1: C14-net -> hv-2
- C4 pad 2: C14-net-1 -> gnd
- C5 pad 1: C15-net -> hv-2
- C5 pad 2: C15-net-1 -> gnd
- C6 pad 1: C16-net -> hv-2
- C6 pad 2: C16-net-1 -> gnd
- C7 pad 1: C17-net -> hv-2
- C7 pad 2: C17-net-1 -> gnd
- C8 pad 1: C18-net-1 -> hv-2
- C8 pad 2: C18-net -> gnd
- C9 pad 1: C19-net -> hv-2
- C9 pad 2: C19-net-1 -> gnd
- U1 pad 11: SDMMC0_CLK_UART5_RTSN_M0_I2C0_SCL_M2_PWM10_M0_GPIO3_A4_d -> SDMMC_CLK_FL
- U1 pad 20: USB_AVDD3V3 -> hv-3
- U1 pad 34: DDR_VDDQ_1 -> VCC_DDR
- U1 pad 35: DDR_VDDQ_2 -> VCC_DDR
- U1 pad 36: DVDD -> hv-2
- U1 pad 38: DDR_PLL_AVDD1V8 -> hv-4
- U1 pad 39: DVDD -> hv-2
- U1 pad 40: DDR_VDDQ_3 -> VCC_DDR
- U1 pad 44: DVDD -> hv-2
- U1 pad 58: DVDD -> hv-2
- U1 pad 6: DVDD -> hv-2
- U1 pad 71: ETH_AVDD3V3 -> hv-3
- U1 pad 73: DVDD -> hv-2
- U1 pad 74: DVDD -> hv-2
- U1 pad 75: DVDD -> hv-2

Commit message: added flash and sd card
Parts:
- added R4: 1kΩ ±1% 62.5mW, atopile:R0402-56259e, F.Cu at (122.2, 51.2)
- added U2: , atopile:WSON-8_L6.0-W5.0-P1.27-BL-EP-5c84f1, F.Cu at (106.6, 164.0)
- added U3: , lib:TF-SMD_TF-01A, F.Cu at (132.2, 51.2)
- moved C1 204.0 mm to (106.6, 124.0)
- moved C10 204.0 mm to (106.6, 94.0)
- moved C11 204.0 mm to (106.6, 84.0)
- moved C12 204.0 mm to (106.6, 74.0)
- moved C13 204.0 mm to (106.6, 124.0)
- moved C14 204.0 mm to (106.6, 54.0)
- moved C15 204.0 mm to (106.6, 64.0)
- moved C16 204.0 mm to (106.6, 44.0)
- moved C18 204.0 mm to (106.6, 24.0)
- moved C19 204.0 mm to (106.6, 114.0)
- moved C2 204.0 mm to (106.6, 114.0)
- moved C20 204.0 mm to (106.6, 94.0)
- moved C21 204.0 mm to (106.6, 34.0)
- moved C22 204.0 mm to (106.6, 74.0)
- moved C23 204.0 mm to (106.6, 104.0)
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Connections:
- net C1-net renamed hv-5
- C1 pad 1: hv-2 -> hv
- C10 pad 1: hv-2 -> hv
- C11 pad 1: hv-2 -> hv
- C12 pad 1: hv-2 -> hv
- C13 pad 2: C1-net-1 -> gnd
- C14 pad 1: hv-3 -> hv-2
- C15 pad 1: hv-3 -> hv-2
- C17 pad 1: C8-net-1 -> C8-net
- C17 pad 2: C8-net -> C8-net-1
- C18 pad 1: C9-net -> C9-net-1
- C18 pad 2: C9-net-1 -> C9-net
- C2 pad 1: hv-2 -> hv
- C20 pad 1: C11-net-1 -> C11-net
- C20 pad 2: C11-net -> C11-net-1
- C21 pad 1: hv-1 -> hv-3
- C22 pad 1: hv-1 -> hv-3
- C3 pad 1: hv-2 -> hv
- C4 pad 1: hv-2 -> hv
- C5 pad 1: hv-2 -> hv
- C6 pad 1: hv-2 -> hv
- C7 pad 1: hv-2 -> hv
- C8 pad 1: hv-2 -> hv
- C9 pad 1: hv-2 -> hv
- L1 pad 2: hv-1 -> hv-3
- R2 pad 2: hv -> hv-1
- U1 pad 20: hv-3 -> hv-2
- U1 pad 36: hv-2 -> hv
- U1 pad 39: hv-2 -> hv
- U1 pad 44: hv-2 -> hv
- U1 pad 58: hv-2 -> hv
- U1 pad 6: hv-2 -> hv
- U1 pad 71: hv-3 -> hv-2
- U1 pad 73: hv-2 -> hv
- U1 pad 74: hv-2 -> hv
- U1 pad 75: hv-2 -> hv

Commit message: fixed errors
Parts:
- added C25: 100nF ±10% 16V X7R, atopile:C0402-b3ef17, F.Cu at (0.00, -80.0)
- added C26: 100nF ±10% 16V X7R, atopile:C0402-b3ef17, F.Cu at (0.00, -60.0)
- added C27: 100nF ±10% 16V X7R, atopile:C0402-b3ef17, F.Cu at (0.00, -40.0)
- added C28: 100nF ±10% 16V X7R, atopile:C0402-b3ef17, F.Cu at (0.00, -30.0)
- added C29: 100nF ±10% 16V X7R, atopile:C0402-b3ef17, F.Cu at (0.00, -100.0)
- added C30: 100nF ±10% 16V X7R, atopile:C0402-b3ef17, F.Cu at (0.00, -110.0)
- added C31: 100nF ±10% 16V X7R, atopile:C0402-b3ef17, F.Cu at (0.00, 0.00)
- added R5: 0Ω 50mW, atopile:R0201-27027e, F.Cu at (0.00, -120.0)
- added R6: 0Ω 50mW, atopile:R0201-27027e, F.Cu at (0.00, -20.0)
- added R7: 0Ω 50mW, atopile:R0201-27027e, F.Cu at (0.00, -90.0)
- added R8: 0Ω 50mW, atopile:R0201-27027e, F.Cu at (0.00, -70.0)
- added R9: 0Ω 50mW, atopile:R0201-27027e, F.Cu at (0.00, -10.0)
- added X1: , atopile:CRYSTAL-SMD_4P-L3.2-W2.5-BL-2-acd8b5, F.Cu at (0.00, -50.0)
Connections:
- net GPIO3_C5_d renamed MIPI_LVDS_RST
- net I2C3_SCL_M1_UART5_TX_M1_PWM11_IR_M2_AUD_DSM_N_GPIO1_D3_d renamed GPIO_D3_d
- net I2C3_SDA_M1_UART5_RX_M1_SPI0_CS1_M0_PWM0_M1_AUD_DSM_P_GPIO1_D2_d renamed GPIO1_D2_d
- net I2C4_SCL_M2_UART5_TX_M2_GPIO3_C7_d renamed MIPI_I2C_SCL
- net I2C4_SDA_M2_UART5_RX_M2_GPIO3_D0_d renamed MIPI_I2C_SDA
- net MIPI_CSI_RX_CK0N_LVDS_RX_CK0N_GPI3_C0_d renamed MIPI_LVDS_CLKN
- net MIPI_CSI_RX_CK0P_LVDS_RX_CK0P_GPI3_C1_d renamed MIPI_LVDS_CLKP
- net MIPI_CSI_RX_CK1N_LVDS_RX_CK1N_GPI3_B2_d renamed GP13_B2_d
- net MIPI_CSI_RX_CK1P_LVDS_RX_CK1P_GPI3_B3_d renamed GP13_B3_d
- net MIPI_CSI_RX_D0N_LVDS_RX_D0N_GPI3_C2_d renamed MIPI_LVDS_D0N
- net MIPI_CSI_RX_D0P_LVDS_RX_D0P_GPI3_C3_d renamed MIPI_LVDS_D0P
- net MIPI_CSI_RX_D1N_LVDS_RX_D1N_GPI3_B6_d renamed MIPI_LVDS_D1N
- net MIPI_CSI_RX_D1P_LVDS_RX_D1P_GPI3_B7_d renamed MIPI_LVDS_D1P
- net MIPI_CSI_RX_D2N_LVDS_RX_D2N_GPI3_B4_d renamed MIPI_LVDS_D2N
- net MIPI_CSI_RX_D3N_LVDS_RX_D3N_GPI3_B0_d renamed MIPI_LVDS_D3N
- net PWM10_M1_UART4_RTSN_M1_GPIO1_C6_d renamed GPIO1_C6_d
- net PWM10_M2_UART5_CTS_M1_UART3_RX_M1_GPIO1_D1_d renamed GPIO1_D1_d
- net PWM11_IR_M1_UART4_CTSN_M1_GPIO1_C7_d renamed GPIO_C7_d
- net PWM2_M2_SPI0_CS0_M0_SDMMC1_D1_M1_GPIO1_C0_d renamed GPIO1_C0_d
- net PWM3_IR_M2_UART5_RTS_M1_UART3_TX_M1_GPIO1_D0_d renamed GPIO_D0_d
- net PWM4_M2_SPI0_CLK_M0_SDMMC1_D0_M1_GPIO1_C1_d renamed GPIO_C1_d
- net PWM5_M2_I2C4_SCL_M1_SDMMC1_CLK_M1_SPI0_MOSI_M0_GPIO1_C2_d renamed GPIO1_C2_d
- net PWM6_M2_I2C4_SDA_M1_SDMMC1_CMD_M1_SPI0_MISO_M0_GPIO1_C3_d renamed GPIO1_C3_d
- net PWM7_IR_M2_MIPI_CLK1_OUT_GPIO3_C6_d renamed GPIO3_C6_d
- net PWM8_M1_UART4_RX_M1_SDMMC1_D3_M1_GPIO1_C4_d renamed GPIO1_C4_d
- net PWM9_M1_UART4_TX_M1_SDMMC1_D2_M1_GPIO1_C5_d renamed GPIO1_C5_d
- net SDMMC0_CMD_UART5_CTS_M0_I2C0_SDA_M2_PWM11_IR_M0_GPIO3_A5_u renamed SDMMC_CMD
- C13 pad 1: hv-5 -> hv-3
- C14 pad 1: hv-2 -> hv-4
- C15 pad 1: hv-2 -> hv-4
- C16 pad 1: C4-net -> C4-net-1
- C16 pad 2: C4-net-1 -> C4-net
- C17 pad 1: C8-net -> C8-net-1
- C17 pad 2: C8-net-1 -> C8-net
- C18 pad 1: C9-net-1 -> C9-net
- C18 pad 2: C9-net -> C9-net-1
- C20 pad 1: C11-net -> C11-net-1
- C20 pad 2: C11-net-1 -> C11-net
- C21 pad 1: hv-3 -> hv-2
- C22 pad 1: hv-3 -> hv-2
- C23 pad 1: hv-4 -> hv-1
- C24 pad 1: hv-4 -> hv-1
- L1 pad 1: hv-4 -> hv-1
- L1 pad 2: hv-3 -> hv-2
- R2 pad 1: hv-4 -> hv-1
- R2 pad 2: hv-1 -> hv-5
- U1 pad 1: MIPI_CLK0_OUT_GPIO3_C4_d -> MIPI_LVDS_MCLK0_FL
- U1 pad 20: hv-2 -> hv-4
- U1 pad 32: FSPI_CS0_GPIO4_B0_u -> FSPI_CS0N
- U1 pad 33: FSPI_CLK_GPIO4_B1_d -> FSPI_CLK
- U1 pad 38: hv-4 -> hv-1
- U1 pad 59: GPIO6_VCC -> hv-4
- U1 pad 7: GPIO4_VCC3V3 -> hv-4
- U1 pad 71: hv-2 -> hv-4
- U1 pad 77: MIPI_CSI_RX_D3P_LVDS_RX_D3P_GPI3_B1_d -> MIPI_LVDS_D2P
- U1 pad 81: MIPI_CSI_RX_D2P_LVDS_RX_D2P_GPI3_B5_d -> MIPI_LVDS_D2P
- U2 pad 1: flash-net-4 -> FSPI_CS0N
- U2 pad 2: flash-net-5 -> FSPI_D1_GPIO4_A3_u
- U2 pad 3: flash-net-7 -> FSPI_D2_GPIO4_A2_u
- U2 pad 4: flash-net -> gnd
- U2 pad 5: flash-net-6 -> FSPI_D0_GPIO4_A4_u
- U2 pad 6: flash-net-1 -> FSPI_D3_GPIO4_A6_u
- U2 pad 7: flash-net-3 -> FSPI_CLK
- U2 pad 8: flash-net-8 -> hv-4
- U2 pad 9: flash-net-2 -> gnd

Commit message: edits
Parts:
- added C32: 100nF ±10% 16V X7R, atopile:C0402-b3ef17, F.Cu at (10.0, 0.00)
- added C33: 100nF ±10% 50V X7R, atopile:C0603-bd72f6, F.Cu at (10.0, -30.0)
- added C34: 100nF ±10% 50V X7R, atopile:C0603-bd72f6, F.Cu at (10.0, -20.0)
- added L2: , atopile:IND-SMD_L3.0-W3.0-a13401, F.Cu at (10.0, -40.0)
- added R10: 200kΩ ±1% 62.5mW, atopile:R0402-56259e, F.Cu at (10.0, -10.0)
- added R11: 100kΩ ±1% 62.5mW, atopile:R0402-56259e, F.Cu at (10.0, -50.0)
- added R12: 4.7kΩ ±1% 62.5mW, atopile:R0402-56259e, F.Cu at (0.00, 0.00)
- added R13: 4.7kΩ ±1% 62.5mW, atopile:R0402-56259e, F.Cu at (0.00, -10.0)
- added U4: , atopile:SOT-23-5_L3.0-W1.7-P0.95-LS2.8-BR-9d80aa, F.Cu at (10.0, -60.0)
- added U5: , lib:USB-C-SMD_KH-TYPE-C-16P, F.Cu at (0.00, -20.0)
- moved C25 178.2 mm to (84.9, 76.7)
- moved C26 178.2 mm to (84.9, 96.7)
- moved C27 178.2 mm to (84.9, 116.7)
- moved C28 178.2 mm to (84.9, 126.7)
- moved C29 178.2 mm to (84.9, 56.7)
- moved C30 178.2 mm to (84.9, 46.7)
- moved C31 178.2 mm to (84.9, 156.7)
- moved R5 178.2 mm to (84.9, 36.7)
- moved R6 178.2 mm to (84.9, 136.7)
- moved R7 178.2 mm to (84.9, 66.7)
- moved R8 178.2 mm to (84.9, 86.7)
- moved R9 178.2 mm to (84.9, 146.7)
- moved X1 178.2 mm to (84.9, 106.7)
- moved U1 39.2 mm to (136.1, 79.8)
Connections:
- C1 pad 1: hv -> hv-2
- C10 pad 1: hv -> hv-2
- C11 pad 1: hv -> hv-2
- C12 pad 1: hv -> hv-2
- C13 pad 1: hv-3 -> hv-1
- C14 pad 1: hv-4 -> hv-5
- C15 pad 1: hv-4 -> hv-5
- C2 pad 1: hv -> hv-2
- C20 pad 1: C11-net-1 -> C11-net
- C20 pad 2: C11-net -> C11-net-1
- C21 pad 1: hv-2 -> hv
- C22 pad 1: hv-2 -> hv
- C23 pad 1: hv-1 -> hv-6
- C24 pad 1: hv-1 -> hv-6
- C27 pad 1: hv-4 -> hv-5
- C28 pad 1: hv-4 -> hv-5
- C3 pad 1: hv -> hv-2
- C30 pad 1: hv-4 -> hv-5
- C31 pad 1: hv-4 -> hv-5
- C4 pad 1: hv -> hv-2
- C5 pad 1: hv -> hv-2
- C6 pad 1: hv -> hv-2
- C7 pad 1: hv -> hv-2
- C8 pad 1: hv -> hv-2
- C9 pad 1: hv -> hv-2
- L1 pad 1: hv-1 -> hv-6
- L1 pad 2: hv-2 -> hv
- R2 pad 1: hv-1 -> hv-6
- R2 pad 2: hv-5 -> hv-4
- R7 pad 1: hv-4 -> hv-5
- R8 pad 1: hv-4 -> hv-5
- U1 pad 20: hv-4 -> hv-5
- U1 pad 36: hv -> hv-2
- U1 pad 38: hv-1 -> hv-6
- U1 pad 39: hv -> hv-2
- U1 pad 44: hv -> hv-2
- U1 pad 58: hv -> hv-2
- U1 pad 59: hv-4 -> hv-5
- U1 pad 6: hv -> hv-2
- U1 pad 7: hv-4 -> hv-5
- U1 pad 71: hv-4 -> hv-5
- U1 pad 73: hv -> hv-2
- U1 pad 74: hv -> hv-2
- U1 pad 75: hv -> hv-2
- U2 pad 8: hv-4 -> hv-5
